File: Kicad/V2/Essaie/Essaie.kicad_sch (KiCad schematic)
At the start: 0 parts

Commit message: pcb_terminé
Parts:
- added U1: ESP32-WROOM-32, RF_Module:ESP32-WROOM-32, symbol RF_Module:ESP32-WROOM-32
- added U2, U3, U4: INA237, Package_SO:TSSOP-10_3x3mm_P0.5mm, symbol Sensor_Energy:INA237
Connections:
- new net: U2.4 (SDA), U3.4 (SDA), U4.4 (SDA)
- new net: U1.20 (SCK/CLK), U2.5 (SCL), U3.5 (SCL), U4.5 (SCL)
- new net: U1.1 (GND), U1.15 (GND), U1.38 (GND), U1.39 (GND), U2.7 (GND), U3.7 (GND), U4.7 (GND)
- new net +BATT: U2.10 (Vin+), U3.10 (Vin+), U4.10 (Vin+)
- new net GND: U2.9 (Vin-), U3.9 (Vin-), U4.9 (Vin-)
Other:
- note added: "LDO NCP737AD"
- title: (none) -> Premier protoype de branchement srage*
