File: Kicad/V5/V5.kicad_sch (KiCad schematic)
At the start: 18 parts, among them J1 Conn_01x02_Pin, U1 ISOM8600DFGR, U2 ISOM8600DFGR, U3 MCP23017-E/SO, U4 ISOM8600DFGR, U5 MIC5283-3.3YME, U7 INA237AIDGSR

Commit message: toutes les fonctions I2C écrite, il faut écrire les fonctions de gestion pure (batterie par batterie)
Parts:
- BT1: footprint Connector_PinHeader_2.54mm:PinHeader_1x02_P2.54mm_Vertical -> Resistor_THT:R_Axial_DIN0207_L6.3mm_D2.5mm_P5.08mm_Vertical
Changed lines of the file:
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@@
       (effects (font (size 1.27 1.27)))
     )
-    (property "Footprint" "Connector_PinHeader_2.54mm:PinHeader_1x02_P2.54mm_Vertical" (at 75.946 154.94 90)
+    (property "Footprint" "Resistor_THT:R_Axial_DIN0207_L6.3mm_D2.5mm_P5.08mm_Vertical" (at 75.946 154.94 90)
       (effects (font (size 1.27 1.27)) hide)
     )
