File: Kicad_projet_salle_blanche/Kicad_projet_salle_blanche.kicad_pcb (KiCad board)
At the start: 2 copper layers, 58.4 x 46.7 mm, 6 parts, among them IC1 HDC3120QDEFRQ1, J1 Conn_01x05_Pin, U2 TPS7A2050PDBVR

Commit message: modif de fin de semaine début du code pour le projet salle blanche
Parts:
- moved J1 1.74 mm to (153.1, 93.5), turned to 0 degrees
Routing:
- net 5V_LDO: track 40.0 -> 46.4 mm
- net SDA: track 14.5 -> 20.6 mm
- net SCL: track 11.8 -> 9.71 mm
Changed lines of the file:
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@@
   (net 31 "unconnected-(U2-N{slash}C-Pad4)")
   (footprint "Connector_JST:JST_AUH_BM05B-AUHKS-GA-TB_1x05-1MP_P1.50mm_Vertical" (layer "F.Cu")
-    (at 153.28 91.74 180)
+    (at 153.12 93.47)
     (descr "JST AUH series connector, BM05B-AUHKS-GA-TB (http://www.jst-mfg.com/product/pdf/eng/eAUH.pdf), generated with kicad-footprint-generator")
     (tags "connector JST AUH vertical")
@@
     (property "ki_keywords" "connector")
     (attr smd)
-    (fp_text reference "J1" (at 0 -3.72) (layer "F.SilkS")
+    (fp_text reference "J1" (at 0 -3.72) (layer "F.SilkS") hide
         (effects (font (size 1 1) (thickness 0.15)))
     )
@@
     (fp_line (start 4.775 -2.075) (end 4.775 2.225)
       (stroke (width 0.1) (type solid)) (layer "F.Fab"))
-    (pad "1" smd roundrect (at -3 -2 180) (size 0.6 1.05) (layers "F.Cu" "F.Paste" "F.Mask") (roundrect_rratio 0.25)
+    (pad "1" smd roundrect (at -3 -2) (size 0.6 1.05) (layers "F.Cu" "F.Paste" "F.Mask") (roundrect_rratio 0.25)
       (net 1 "GND") (pinfunction "Pin_1") (pintype "passive"))
-    (pad "2" smd roundrect (at -1.5 -2 180) (size 0.6 1.05) (layers "F.Cu" "F.Paste" "F.Mask") (roundrect_rratio 0.25)
+    (pad "2" smd roundrect (at -1.5 -2) (size 0.6 1.05) (layers "F.Cu" "F.Paste" "F.Mask") (roundrect_rratio 0.25)
       (net 1 "GND") (pinfunction "Pin_2") (pintype "passive"))
-    (pad "3" smd roundrect (at 0 -2 180) (size 0.6 1.05) (layers "F.Cu" "F.Paste" "F.Mask") (roundrect_rratio 0.25)
+    (pad "3" smd roundrect (at 0 -2) (size 0.6 1.05) (layers "F.Cu" "F.Paste" "F.Mask") (roundrect_rratio 0.25)
       (net 4 "SCL") (pinfunction "Pin_3") (pintype "passive"))
-    (pad "4" smd roundrect (at 1.5 -2 180) (size 0.6 1.05) (layers "F.Cu" "F.Paste" "F.Mask") (roundrect_rratio 0.25)
+    (pad "4" smd roundrect (at 1.5 -2) (size 0.6 1.05) (layers "F.Cu" "F.Paste" "F.Mask") (roundrect_rratio 0.25)
       (net 5 "SDA") (pinfunction "Pin_4") (pintype "passive"))
-    (pad "5" smd roundrect (at 3 -2 180) (size 0.6 1.05) (layers "F.Cu" "F.Paste" "F.Mask") (roundrect_rratio 0.25)
+    (pad "5" smd roundrect (at 3 -2) (size 0.6 1.05) (layers "F.Cu" "F.Paste" "F.Mask") (roundrect_rratio 0.25)
       (net 2 "5V_LDO") (pinfunction "Pin_5") (pintype "passive"))
-    (pad "MP" smd roundrect (at -4.45 1.8 180) (size 0.6 1.45) (layers "F.Cu" "F.Paste" "F.Mask") (roundrect_rratio 0.25))
-    (pad "MP" smd roundrect (at 4.45 1.8 180) (size 0.6 1.45) (layers "F.Cu" "F.Paste" "F.Mask") (roundrect_rratio 0.25))
+    (pad "MP" smd roundrect (at -4.45 1.8) (size 0.6 1.45) (layers "F.Cu" "F.Paste" "F.Mask") (roundrect_rratio 0.25))
+    (pad "MP" smd roundrect (at 4.45 1.8) (size 0.6 1.45) (layers "F.Cu" "F.Paste" "F.Mask") (roundrect_rratio 0.25))
     (model "${KICAD7_3DMODEL_DIR}/Connector_JST.3dshapes/JST_AUH_BM05B-AUHKS-GA-TB_1x05-1MP_P1.50mm_Vertical.wrl"
       (offset (xyz 0 0 0))
@@
   (segment (start 119.09 94.15) (end 124.16 94.15) (width 0.5) (layer "F.Cu") (net 2))
   (segment (start 136.53 91.61) (end 136.53 91.51) (width 0.5) (layer "F.Cu") (net 2))
-  (segment (start 133.99 94.15) (end 149.87 94.15) (width 0.5) (layer "F.Cu") (net 2))
   (segment (start 126.22 92.09) (end 125.69 92.62) (width 0.2) (layer "F.Cu") (net 2))
   (segment (start 124.16 94.15) (end 125.69 92.62) (width 0.5) (layer "F.Cu") (net 2))
+  (segment (start 138.465 94.095) (end 136.13 91.76) (width 0.5) (layer "F.Cu") (net 2))
   (segment (start 133.99 94.15) (end 135.585 92.555) (width 0.5) (layer "F.Cu") (net 2))
   (segment (start 135.585 92.555) (end 136.53 91.61) (width 0.5) (layer "F.Cu") (net 2))
+  (segment (start 156.12 91.47) (end 156.12 92.52) (width 0.5) (layer "F.Cu") (net 2))
   (segment (start 135.585 92.555) (end 136.13 92.01) (width 0.5) (layer "F.Cu") (net 2))
-  (segment (start 149.87 94.15) (end 150.28 93.74) (width 0.5) (layer "F.Cu") (net 2))
+  (segment (start 156.12 92.52) (end 154.545 94.095) (width 0.5) (layer "F.Cu") (net 2))
+  (segment (start 154.545 94.095) (end 138.465 94.095) (width 0.5) (layer "F.Cu") (net 2))
   (segment (start 136.13 92.01) (end 136.13 91.51) (width 0.5) (layer "F.Cu") (net 2))
   (segment (start 124.16 94.15) (end 133.99 94.15) (width 0.5) (layer "F.Cu") (net 2))
+  (segment (start 136.13 91.76) (end 136.13 91.51) (width 0.5) (layer "F.Cu") (net 2))
   (segment (start 126.35 87.54) (end 127.33 87.54) (width 0.5) (layer "F.Cu") (net 3))
   (segment (start 127.72 88.86) (end 127.72 87.93) (width 0.2) (layer "F.Cu") (net 3))
@@
   (segment (start 118.33 66.32) (end 118.33 86.375) (width 0.5) (layer "F.Cu") (net 3))
   (segment (start 127.33 87.54) (end 127.44 87.65) (width 0.5) (layer "F.Cu") (net 3))
-  (segment (start 153.28 93.74) (end 153.28 82.080374) (width 0.5) (layer "F.Cu") (net 4))
   (segment (start 153.28 82.080374) (end 153.370374 81.99) (width 0.5) (layer "F.Cu") (net 4))
-  (segment (start 151.340374 87.58) (end 145.750374 81.99) (width 0.5) (layer "F.Cu") (net 5))
-  (segment (start 151.78 93.74) (end 151.78 87.62) (width 0.5) (layer "F.Cu") (net 5))
-  (segment (start 151.78 87.62) (end 151.74 87.58) (width 0.5) (layer "F.Cu") (net 5))
-  (segment (start 151.74 87.58) (end 151.340374 87.58) (width 0.5) (layer "F.Cu") (net 5))
+  (segment (start 153.370374 91.219626) (end 153.12 91.47) (width 0.5) (layer "F.Cu") (net 4))
+  (segment (start 153.370374 81.99) (end 153.370374 91.219626) (width 0.5) (layer "F.Cu") (net 4))
+  (segment (start 152.96 93.18) (end 152.96 93.13) (width 0.5) (layer "F.Cu") (net 5))
+  (segment (start 145.750374 91.880374) (end 147.05 93.18) (width 0.5) (layer "F.Cu") (net 5))
+  (segment (start 147.05 93.18) (end 152.96 93.18) (width 0.5) (layer "F.Cu") (net 5))
+  (segment (start 152.96 93.13) (end 154.62 91.47) (width 0.5) (layer "F.Cu") (net 5))
+  (segment (start 145.750374 81.99) (end 145.750374 91.880374) (width 0.5) (layer "F.Cu") (net 5))
+  (segment (start 154.62 92.08) (end 154.62 91.47) (width 0.2) (layer "F.Cu") (net 5))
   (segment (start 129.370374 83.39) (end 132.96 83.39) (width 0.5) (layer "F.Cu") (net 10))
   (segment (start 127.970374 81.99) (end 129.370374 83.39) (width 0.5) (layer "F.Cu") (net 10))

Commit message: 4 pcb terminé
Parts:
- removed IC1: HDC3120QDEFRQ1, TPS7...:SON50P250X250X80-9N-D
- added G***: LOGO, ESP32_Footprints:ETS, F.Cu at (139.3, 69.5)
- added U3: SHT40-CD1B-R3, Esp:U_SHT3_SEN, F.Cu at (142.0, 88.6)
- J1: footprint Connector_JST:JST_AUH_BM05B-AUHKS-GA-TB_1x05-1MP_P1.50mm_Vertical -> Connector_PinHeader_2.54mm:PinHeader_1x05_P2.54mm_Vertical
- U1: footprint ESP32_Footprints:ESP32_30pin -> Esp:esp32_devkit_v1_doit
- U2: value TPS7A2050PDBVR -> TLV75533PDYDR; footprint TPS7...:SON50P250X250X80-9N-D -> Esp:DBV0005A-MFG
- moved U1 18.4 mm to (120.0, 68.8), turned to -90 degrees
- moved J1 6.02 mm to (158.6, 90.9), turned to -90 degrees
- moved U2 0.30 mm to (127.3, 90.2)
- moved C1 0.12 mm to (114.1, 94.0)
Routing:
- net SCL: track 9.71 -> 40.4 mm
- net SDA: track 20.6 -> 41.2 mm
- net ADC_TEMP: track 13.6 -> 0.00 mm
- net ADC_HUM: track 13.2 -> 0.00 mm
- net GND: track 4.06 -> 1.72 mm, vias 0 -> 4
- net 5V: track 43.1 -> 44.9 mm
- net 5V_LDO: track 46.4 -> 47.2 mm
- added copper zone on B.Cu, net GND
Other:
- outline, holes or cut-outs redrawn
- board text removed: "LDO"
- board text removed: "RH"
