File: Kicad/V6/V6/V6.kicad_pcb (KiCad board)
At the start: 2 copper layers, 75 x 119.2 mm, 65 parts, among them J1 Conn_01x05_Pin, J2 Conn_01x02_Pin, J3 Conn_01x02_Pin, J39 Conn_01x02_Pin, J4 Conn_01x02_Pin, J41 Conn_01x02_Pin, J42 Conn_01x02_Pin, J43 Conn_01x02_Pin, J44 Conn_01x02_Pin, J45 Conn_01x02_Pin, J5 Conn_01x02_Pin, J6 Conn_01x02_Pin, J7 Conn_01x02_Pin, U1 WPME-FDSM_SIP-3, U10 ISOM8600DFGR, U11 ISOM8600DFGR, U12 ISOM8600DFGR, U13 ISOM8600DFGR, U14 ISOM8600DFGR, U15 ISOM8600DFGR, U3 MCP23017-E/SO, U31 ISOM8600DFGR, U32 ISOM8600DFGR, U33 ISOM8600DFGR, U34 ISOM8600DFGR, U35 ISOM8600DFGR, U36 ISOM8600DFGR, U4 ISOM8600DFGR, U5 TLV75533PDYDR, U7 INA237AIDGSR, U8 ISOM8600DFGR, U9 ISOM8600DFGR

Commit message: Pojet batterie fonctionne, plus création du readme
Connections:
- U6 pad 10: temp_7 -> temp_3
- U6 pad 11: temp_8 -> temp_2
- U6 pad 12: temp_9 -> temp_1
- U6 pad 13: temp_10 -> temp_base
- U6 pad 3: temp_base -> temp_10
- U6 pad 4: temp_1 -> temp_9
- U6 pad 5: temp_2 -> temp_8
- U6 pad 6: temp_3 -> temp_7
- U6 pad 7: temp_4 -> temp_6
- U6 pad 9: temp_6 -> temp_4
Routing:
- net 5V: track 118.1 -> 153.2 mm
Changed lines of the file:
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@@
     (fp_circle (center 11.7 43.46) (end 13.2 43.46)
       (stroke (width 0.12) (type solid)) (fill none) (layer "F.SilkS"))
-    (pad "1" thru_hole rect (at -12.7 0) (size 1.524 1.524) (drill 0.762) (layers "*.Cu" "*.Mask")
+    (pad "1" thru_hole rect (at -12.7 35.56 180) (size 1.524 1.524) (drill 0.762) (layers "*.Cu" "*.Mask")
       (net 65 "5V") (pinfunction "VIN") (pintype "power_out"))
-    (pad "2" thru_hole circle (at -12.7 2.54) (size 1.524 1.524) (drill 0.762) (layers "*.Cu" "*.Mask")
+    (pad "2" thru_hole circle (at -12.7 33.02 180) (size 1.524 1.524) (drill 0.762) (layers "*.Cu" "*.Mask")
       (net 2 "GND") (pinfunction "GND") (pintype "bidirectional"))
-    (pad "3" thru_hole circle (at -12.7 5.08) (size 1.524 1.524) (drill 0.762) (layers "*.Cu" "*.Mask")
-      (net 16 "temp_base") (pinfunction "GPIO13") (pintype "bidirectional"))
-    (pad "4" thru_hole circle (at -12.7 7.62) (size 1.524 1.524) (drill 0.762) (layers "*.Cu" "*.Mask")
-      (net 10 "temp_1") (pinfunction "GPIO12") (pintype "bidirectional"))
-    (pad "5" thru_hole circle (at -12.7 10.16) (size 1.524 1.524) (drill 0.762) (layers "*.Cu" "*.Mask")
-      (net 11 "temp_2") (pinfunction "GPIO14") (pintype "bidirectional"))
-    (pad "6" thru_hole circle (at -12.7 12.7) (size 1.524 1.524) (drill 0.762) (layers "*.Cu" "*.Mask")
-      (net 12 "temp_3") (pinfunction "GPIO27") (pintype "bidirectional"))
-    (pad "7" thru_hole circle (at -12.7 15.24) (size 1.524 1.524) (drill 0.762) (layers "*.Cu" "*.Mask")
-      (net 13 "temp_4") (pinfunction "GPIO26") (pintype "bidirectional"))
-    (pad "8" thru_hole circle (at -12.7 17.78) (size 1.524 1.524) (drill 0.762) (layers "*.Cu" "*.Mask")
+    (pad "3" thru_hole circle (at -12.7 30.48 180) (size 1.524 1.524) (drill 0.762) (layers "*.Cu" "*.Mask")
+      (net 58 "temp_10") (pinfunction "GPIO13") (pintype "bidirectional"))
+    (pad "4" thru_hole circle (at -12.7 27.94 180) (size 1.524 1.524) (drill 0.762) (layers "*.Cu" "*.Mask")
+      (net 57 "temp_9") (pinfunction "GPIO12") (pintype "bidirectional"))
+    (pad "5" thru_hole circle (at -12.7 25.4 180) (size 1.524 1.524) (drill 0.762) (layers "*.Cu" "*.Mask")
+      (net 56 "temp_8") (pinfunction "GPIO14") (pintype "bidirectional"))
+    (pad "6" thru_hole circle (at -12.7 22.86 180) (size 1.524 1.524) (drill 0.762) (layers "*.Cu" "*.Mask")
+      (net 55 "temp_7") (pinfunction "GPIO27") (pintype "bidirectional"))
+    (pad "7" thru_hole circle (at -12.7 20.32 180) (size 1.524 1.524) (drill 0.762) (layers "*.Cu" "*.Mask")
+      (net 54 "temp_6") (pinfunction "GPIO26") (pintype "bidirectional"))
+    (pad "8" thru_hole circle (at -12.7 17.78 180) (size 1.524 1.524) (drill 0.762) (layers "*.Cu" "*.Mask")
       (net 53 "temp_5") (pinfunction "GPIO25") (pintype "bidirectional"))
-    (pad "9" thru_hole circle (at -12.7 20.32) (size 1.524 1.524) (drill 0.762) (layers "*.Cu" "*.Mask")
-      (net 54 "temp_6") (pinfunction "GPIO33") (pintype "bidirectional"))
-    (pad "10" thru_hole circle (at -12.7 22.86) (size 1.524 1.524) (drill 0.762) (layers "*.Cu" "*.Mask")
-      (net 55 "temp_7") (pinfunction "GPIO32") (pintype "bidirectional"))
-    (pad "11" thru_hole circle (at -12.7 25.4) (size 1.524 1.524) (drill 0.762) (layers "*.Cu" "*.Mask")
-      (net 56 "temp_8") (pinfunction "GPIO35") (pintype "bidirectional"))
-    (pad "12" thru_hole circle (at -12.7 27.94) (size 1.524 1.524) (drill 0.762) (layers "*.Cu" "*.Mask")
-      (net 57 "temp_9") (pinfunction "GPIO34") (pintype "bidirectional"))
-    (pad "13" thru_hole circle (at -12.7 30.48) (size 1.524 1.524) (drill 0.762) (layers "*.Cu" "*.Mask")
-      (net 58 "temp_10") (pinfunction "GPIO39") (pintype "bidirectional"))
-    (pad "14" thru_hole circle (at -12.7 33.02) (size 1.524 1.524) (drill 0.762) (layers "*.Cu" "*.Mask")
+    (pad "9" thru_hole circle (at -12.7 15.24 180) (size 1.524 1.524) (drill 0.762) (layers "*.Cu" "*.Mask")
+      (net 13 "temp_4") (pinfunction "GPIO33") (pintype "bidirectional"))
+    (pad "10" thru_hole circle (at -12.7 12.7 180) (size 1.524 1.524) (drill 0.762) (layers "*.Cu" "*.Mask")
+      (net 12 "temp_3") (pinfunction "GPIO32") (pintype "bidirectional"))
+    (pad "11" thru_hole circle (at -12.7 10.16 180) (size 1.524 1.524) (drill 0.762) (layers "*.Cu" "*.Mask")
+      (net 11 "temp_2") (pinfunction "GPIO35") (pintype "bidirectional"))
+    (pad "12" thru_hole circle (at -12.7 7.62 180) (size 1.524 1.524) (drill 0.762) (layers "*.Cu" "*.Mask")
+      (net 10 "temp_1") (pinfunction "GPIO34") (pintype "bidirectional"))
+    (pad "13" thru_hole circle (at -12.7 5.08 180) (size 1.524 1.524) (drill 0.762) (layers "*.Cu" "*.Mask")
+      (net 16 "temp_base") (pinfunction "GPIO39") (pintype "bidirectional"))
+    (pad "14" thru_hole circle (at -12.7 2.54 180) (size 1.524 1.524) (drill 0.762) (layers "*.Cu" "*.Mask")
       (net 40 "unconnected-(U6-GPIO36-Pad14)") (pinfunction "GPIO36") (pintype "bidirectional+no_connect"))
-    (pad "15" thru_hole circle (at -12.7 35.56) (size 1.524 1.524) (drill 0.762) (layers "*.Cu" "*.Mask")
+    (pad "15" thru_hole circle (at -12.7 0 180) (size 1.524 1.524) (drill 0.762) (layers "*.Cu" "*.Mask")
       (net 41 "unconnected-(U6-EN-Pad15)") (pinfunction "EN") (pintype "bidirectional+no_connect"))
     (pad "16" thru_hole circle (at 12.7 35.56) (size 1.524 1.524) (drill 0.762) (layers "*.Cu" "*.Mask")
@@
   (segment (start 201.6619 58.815) (end 199.435 58.815) (width 0.7) (layer "F.Cu") (net 39))
   (segment (start 205.2169 62.37) (end 201.6619 58.815) (width 0.7) (layer "F.Cu") (net 39))
+  (segment (start 194.81 92.11) (end 195.1 92.11) (width 0.7) (layer "B.Cu") (net 41))
   (segment (start 230.66 126.405) (end 230.4 126.145) (width 0.7) (layer "F.Cu") (net 50))
   (segment (start 230.66 131.03) (end 230.66 126.405) (width 0.7) (layer "F.Cu") (net 50))
@@
   (via (at 222.56 36.015) (size 1) (drill 0.5) (layers "F.Cu" "B.Cu") (net 65))
   (segment (start 227.99 30.26) (end 226.686 31.564) (width 0.7) (layer "B.Cu") (net 65))
-  (segment (start 193.19 90.49) (end 194.81 92.11) (width 0.7) (layer "B.Cu") (net 65))
-  (segment locked (start 231.83 69.119189) (end 231.83 34.1) (width 0.7) (layer "B.Cu") (net 65))
-  (segment (start 226.686 31.564) (end 226.686 31.889) (width 0.7) (layer "B.Cu") (net 65))
-  (segment (start 216.20774 84.741449) (end 194.988551 84.741449) (width 0.7) (layer "B.Cu") (net 65))
-  (segment (start 194.988551 84.741449) (end 193.19 86.54) (width 0.7) (layer "B.Cu") (net 65))
-  (segment (start 231.83 34.1) (end 227.99 30.26) (width 0.7) (layer "B.Cu") (net 65))
+  (segment (start 216.20774 84.741449) (end 196.094631 84.741449) (width 0.7) (layer "B.Cu") (net 65))
   (segment (start 231.83 69.119189) (end 216.20774 84.741449) (width 0.7) (layer "B.Cu") (net 65))
+  (segment (start 196.094631 84.741449) (end 192.81 88.02608) (width 0.7) (layer "B.Cu") (net 65))
+  (segment (start 192.81 125.38) (end 195.1 127.67) (width 0.7) (layer "B.Cu") (net 65))
+  (segment (start 226.686 31.564) (end 226.686 31.889) (width 0.7) (layer "B.Cu") (net 65))
+  (segment (start 227.99 30.26) (end 231.83 34.1) (width 0.7) (layer "B.Cu") (net 65))
+  (segment (start 231.83 34.1) (end 231.83 69.119189) (width 0.7) (layer "B.Cu") (net 65))
+  (segment (start 192.81 88.02608) (end 192.81 125.38) (width 0.7) (layer "B.Cu") (net 65))
   (segment (start 226.686 31.889) (end 222.56 36.015) (width 0.7) (layer "B.Cu") (net 65))
-  (segment (start 193.19 86.54) (end 193.19 90.49) (width 0.7) (layer "B.Cu") (net 65))
-  (segment (start 194.81 92.11) (end 195.1 92.11) (width 0.7) (layer "B.Cu") (net 65))
   (segment (start 220.5 127.67) (end 221.93 127.67) (width 0.7) (layer "F.Cu") (net 66))
   (segment (start 225.22 130.96) (end 225.22 134.8) (width 0.7) (layer "F.Cu") (net 66))
