File: Kicad_esp_maitre_salle_blanche/Kicad_esp_maitre_salle_blanche/Kicad_esp_maitre_salle_blanche.kicad_pcb (KiCad board)
At the start: 2 copper layers, 58.4 x 46.7 mm, 8 parts, among them J1 Conn_01x05_Pin, J2 Conn_01x04_Pin, U2 TLV75533PDYDR, U3 SHT40-CD1B-R3

Commit message: Pojet batterie fonctionne, plus création du readme
Routing:
- net 5V: track 43.9 -> 73.6 mm
- net SDA: track 54.8 -> 53.7 mm
Changed lines of the file:
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@@
       (outputformat 1)
       (mirror false)
-      (drillshape 1)
+      (drillshape 0)
       (scaleselection 1)
-      (outputdirectory "")
+      (outputdirectory "../Percage, salle blanche/")
     )
   )
@@
     (fp_circle (center 11.7 4.04) (end 13.2 4.04)
       (stroke (width 0.12) (type solid)) (fill none) (layer "B.SilkS"))
-    (pad "1" thru_hole rect (at -12.7 0 270) (size 1.524 1.524) (drill 0.762) (layers "*.Cu" "*.Mask")
+    (pad "1" thru_hole rect (at -12.7 -35.56 90) (size 1.524 1.524) (drill 0.762) (layers "*.Cu" "*.Mask")
       (net 3 "5V") (pinfunction "VIN") (pintype "power_out"))
-    (pad "2" thru_hole circle (at -12.7 -2.54 270) (size 1.524 1.524) (drill 0.762) (layers "*.Cu" "*.Mask")
+    (pad "2" thru_hole circle (at -12.7 -33.02 90) (size 1.524 1.524) (drill 0.762) (layers "*.Cu" "*.Mask")
       (net 1 "GND") (pinfunction "GND") (pintype "bidirectional"))
-    (pad "3" thru_hole circle (at -12.7 -5.08 270) (size 1.524 1.524) (drill 0.762) (layers "*.Cu" "*.Mask")
+    (pad "3" thru_hole circle (at -12.7 -30.48 90) (size 1.524 1.524) (drill 0.762) (layers "*.Cu" "*.Mask")
       (net 6 "unconnected-(U1-GPIO13-Pad3)") (pinfunction "GPIO13") (pintype "bidirectional+no_connect"))
-    (pad "4" thru_hole circle (at -12.7 -7.62 270) (size 1.524 1.524) (drill 0.762) (layers "*.Cu" "*.Mask")
+    (pad "4" thru_hole circle (at -12.7 -27.94 90) (size 1.524 1.524) (drill 0.762) (layers "*.Cu" "*.Mask")
       (net 7 "unconnected-(U1-GPIO12-Pad4)") (pinfunction "GPIO12") (pintype "bidirectional+no_connect"))
-    (pad "5" thru_hole circle (at -12.7 -10.16 270) (size 1.524 1.524) (drill 0.762) (layers "*.Cu" "*.Mask")
+    (pad "5" thru_hole circle (at -12.7 -25.4 90) (size 1.524 1.524) (drill 0.762) (layers "*.Cu" "*.Mask")
       (net 8 "unconnected-(U1-GPIO14-Pad5)") (pinfunction "GPIO14") (pintype "bidirectional+no_connect"))
-    (pad "6" thru_hole circle (at -12.7 -12.7 270) (size 1.524 1.524) (drill 0.762) (layers "*.Cu" "*.Mask")
+    (pad "6" thru_hole circle (at -12.7 -22.86 90) (size 1.524 1.524) (drill 0.762) (layers "*.Cu" "*.Mask")
       (net 9 "unconnected-(U1-GPIO27-Pad6)") (pinfunction "GPIO27") (pintype "bidirectional+no_connect"))
-    (pad "7" thru_hole circle (at -12.7 -15.24 270) (size 1.524 1.524) (drill 0.762) (layers "*.Cu" "*.Mask")
+    (pad "7" thru_hole circle (at -12.7 -20.32 90) (size 1.524 1.524) (drill 0.762) (layers "*.Cu" "*.Mask")
       (net 29 "unconnected-(U1-GPIO26-Pad7)") (pinfunction "GPIO26") (pintype "bidirectional+no_connect"))
-    (pad "8" thru_hole circle (at -12.7 -17.78 270) (size 1.524 1.524) (drill 0.762) (layers "*.Cu" "*.Mask")
+    (pad "8" thru_hole circle (at -12.7 -17.78 90) (size 1.524 1.524) (drill 0.762) (layers "*.Cu" "*.Mask")
       (net 30 "unconnected-(U1-GPIO25-Pad8)") (pinfunction "GPIO25") (pintype "bidirectional+no_connect"))
-    (pad "9" thru_hole circle (at -12.7 -20.32 270) (size 1.524 1.524) (drill 0.762) (layers "*.Cu" "*.Mask")
+    (pad "9" thru_hole circle (at -12.7 -15.24 90) (size 1.524 1.524) (drill 0.762) (layers "*.Cu" "*.Mask")
       (net 12 "unconnected-(U1-GPIO33-Pad9)") (pinfunction "GPIO33") (pintype "bidirectional+no_connect"))
-    (pad "10" thru_hole circle (at -12.7 -22.86 270) (size 1.524 1.524) (drill 0.762) (layers "*.Cu" "*.Mask")
+    (pad "10" thru_hole circle (at -12.7 -12.7 90) (size 1.524 1.524) (drill 0.762) (layers "*.Cu" "*.Mask")
       (net 13 "unconnected-(U1-GPIO32-Pad10)") (pinfunction "GPIO32") (pintype "bidirectional+no_connect"))
-    (pad "11" thru_hole circle (at -12.7 -25.4 270) (size 1.524 1.524) (drill 0.762) (layers "*.Cu" "*.Mask")
+    (pad "11" thru_hole circle (at -12.7 -10.16 90) (size 1.524 1.524) (drill 0.762) (layers "*.Cu" "*.Mask")
       (net 14 "unconnected-(U1-GPIO35-Pad11)") (pinfunction "GPIO35") (pintype "bidirectional+no_connect"))
-    (pad "12" thru_hole circle (at -12.7 -27.94 270) (size 1.524 1.524) (drill 0.762) (layers "*.Cu" "*.Mask")
+    (pad "12" thru_hole circle (at -12.7 -7.62 90) (size 1.524 1.524) (drill 0.762) (layers "*.Cu" "*.Mask")
       (net 15 "unconnected-(U1-GPIO34-Pad12)") (pinfunction "GPIO34") (pintype "bidirectional+no_connect"))
-    (pad "13" thru_hole circle (at -12.7 -30.48 270) (size 1.524 1.524) (drill 0.762) (layers "*.Cu" "*.Mask")
+    (pad "13" thru_hole circle (at -12.7 -5.08 90) (size 1.524 1.524) (drill 0.762) (layers "*.Cu" "*.Mask")
       (net 16 "unconnected-(U1-GPIO39-Pad13)") (pinfunction "GPIO39") (pintype "bidirectional+no_connect"))
-    (pad "14" thru_hole circle (at -12.7 -33.02 270) (size 1.524 1.524) (drill 0.762) (layers "*.Cu" "*.Mask")
+    (pad "14" thru_hole circle (at -12.7 -2.54 90) (size 1.524 1.524) (drill 0.762) (layers "*.Cu" "*.Mask")
       (net 17 "unconnected-(U1-GPIO36-Pad14)") (pinfunction "GPIO36") (pintype "bidirectional+no_connect"))
-    (pad "15" thru_hole circle (at -12.7 -35.56 270) (size 1.524 1.524) (drill 0.762) (layers "*.Cu" "*.Mask")
+    (pad "15" thru_hole circle (at -12.7 0 90) (size 1.524 1.524) (drill 0.762) (layers "*.Cu" "*.Mask")
       (net 18 "unconnected-(U1-EN-Pad15)") (pinfunction "EN") (pintype "bidirectional+no_connect"))
     (pad "16" thru_hole circle (at 12.7 -35.56 270) (size 1.524 1.524) (drill 0.762) (layers "*.Cu" "*.Mask")
@@
   (segment (start 141.800126 86.130126) (end 141.61 85.94) (width 0.2) (layer "F.Cu") (net 2))
   (segment (start 165.22 90.48) (end 163.54 88.8) (width 0.5) (layer "F.Cu") (net 2))
-  (segment (start 119.27 80.54) (end 118.058 81.752) (width 0.5) (layer "F.Cu") (net 3))
+  (segment (start 154.83 57.21) (end 154.83 66.428592) (width 0.5) (layer "F.Cu") (net 3))
   (segment (start 127.680002 87.27) (end 128.220002 87.81) (width 0.5) (layer "F.Cu") (net 3))
+  (segment (start 154.86 66.458592) (end 154.86 70.45) (width 0.5) (layer "F.Cu") (net 3))
+  (segment (start 154.86 70.45) (end 148.43 76.88) (width 0.5) (layer "F.Cu") (net 3))
   (segment (start 124.73 87.27) (end 126.32 88.86) (width 0.5) (layer "F.Cu") (net 3))
   (segment (start 128.220002 87.81) (end 128.220002 88.86) (width 0.5) (layer "F.Cu") (net 3))
+  (segment (start 148.43 76.88) (end 122.93 76.88) (width 0.5) (layer "F.Cu") (net 3))
+  (segment (start 154.83 66.428592) (end 154.86 66.458592) (width 0.5) (layer "F.Cu") (net 3))
+  (segment (start 118.058 86.103) (end 119.225 87.27) (width 0.5) (layer "F.Cu") (net 3))
   (segment (start 124.36 87.27) (end 124.73 87.27) (width 0.5) (layer "F.Cu") (net 3))
-  (segment (start 119.27 57.21) (end 119.27 80.54) (width 0.5) (layer "F.Cu") (net 3))
+  (segment (start 119.225 87.27) (end 124.36 87.27) (width 0.5) (layer "F.Cu") (net 3))
+  (segment (start 124.36 87.27) (end 127.680002 87.27) (width 0.5) (layer "F.Cu") (net 3))
+  (segment (start 122.93 76.88) (end 118.058 81.752) (width 0.5) (layer "F.Cu") (net 3))
   (segment (start 118.058 81.752) (end 118.058 86.103) (width 0.5) (layer "F.Cu") (net 3))
-  (segment (start 119.225 87.27) (end 124.36 87.27) (width 0.5) (layer "F.Cu") (net 3))
-  (segment (start 118.058 86.103) (end 119.225 87.27) (width 0.5) (layer "F.Cu") (net 3))
-  (segment (start 124.36 87.27) (end 127.680002 87.27) (width 0.5) (layer "F.Cu") (net 3))
   (segment (start 152.895 88.6) (end 152.895 87.397919) (width 0.5) (layer "F.Cu") (net 4))
   (segment (start 152.895 87.397919) (end 149.987081 84.49) (width 0.5) (layer "F.Cu") (net 4))
@@
   (segment (start 150.355 86.594626) (end 150.355 88.6) (width 0.5) (layer "F.Cu") (net 5))
   (segment (start 151.76 93.13) (end 161.75 93.13) (width 0.5) (layer "B.Cu") (net 5))
-  (segment (start 135.722 82.107973) (end 135.722 83.572) (width 0.5) (layer "B.Cu") (net 5))
-  (segment (start 129.43 82.61) (end 130.642 81.398) (width 0.5) (layer "B.Cu") (net 5))
-  (segment (start 135.722 83.572) (end 137.39 85.24) (width 0.5) (layer "B.Cu") (net 5))
+  (segment (start 129.43 82.61) (end 129.43 83.9) (width 0.5) (layer "B.Cu") (net 5))
+  (segment (start 149 85.24) (end 150.355 86.595) (width 0.5) (layer "B.Cu") (net 5))
   (segment (start 161.75 93.13) (end 163.54 91.34) (width 0.5) (layer "B.Cu") (net 5))
-  (segment (start 130.642 81.398) (end 135.012027 81.398) (width 0.5) (layer "B.Cu") (net 5))
-  (segment (start 135.012027 81.398) (end 135.722 82.107973) (width 0.5) (layer "B.Cu") (net 5))
   (segment (start 150.355 86.595) (end 150.355 88.6) (width 0.5) (layer "B.Cu") (net 5))
-  (segment (start 149 85.24) (end 150.355 86.595) (width 0.5) (layer "B.Cu") (net 5))
+  (segment (start 130.77 85.24) (end 149 85.24) (width 0.5) (layer "B.Cu") (net 5))
+  (segment (start 129.43 83.9) (end 130.77 85.24) (width 0.5) (layer "B.Cu") (net 5))
   (segment (start 150.355 91.725) (end 150.355 88.6) (width 0.5) (layer "B.Cu") (net 5))
-  (segment (start 137.39 85.24) (end 149 85.24) (width 0.5) (layer "B.Cu") (net 5))
   (segment (start 151.76 93.13) (end 150.355 91.725) (width 0.5) (layer "B.Cu") (net 5))
   (zone (net 1) (net_name "GND") (layers "F&B.Cu") (hatch edge 0.5)
