File: Kicad_esp_maitre_salle_blanche/Kicad_esp_maitre_salle_blanche/Kicad_esp_maitre_salle_blanche.kicad_pcb (KiCad board)
At the start: 2 copper layers, 58.4 x 46.7 mm, 8 parts, among them J1 Conn_01x05_Pin, J2 Conn_01x04_Pin, U2 TLV75533PDYDR, U3 SHT40-CD1B-R3

Commit message: Commit finale
Routing:
- net 5V_LDO: track 77.2 -> 72.1 mm
- net SCL: track 50.9 -> 48.6 mm
Changed lines of the file:
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@@
   (setup
     (pad_to_mask_clearance 0)
+    (grid_origin 140.92 87.47)
     (pcbplotparams
       (layerselection 0x00010fc_ffffffff)
@@
   (segment (start 127.58 94.15) (end 128.220002 93.509998) (width 0.5) (layer "F.Cu") (net 2))
   (segment (start 138.465 94.095) (end 138.465 85.725) (width 0.5) (layer "F.Cu") (net 2))
-  (segment (start 141.800126 87.3816) (end 141.800126 86.130126) (width 0.2) (layer "F.Cu") (net 2))
   (segment (start 147.815 91.485) (end 147.815 88.6) (width 0.5) (layer "F.Cu") (net 2))
-  (segment (start 138.88 85.31) (end 140.98 85.31) (width 0.5) (layer "F.Cu") (net 2))
   (segment (start 145.15 94.15) (end 146.48 95.48) (width 0.5) (layer "F.Cu") (net 2))
   (segment (start 165.22 95.48) (end 165.22 90.48) (width 0.5) (layer "F.Cu") (net 2))
   (segment (start 128.220002 93.509998) (end 128.220002 91.46) (width 0.5) (layer "F.Cu") (net 2))
-  (segment (start 138.465 85.725) (end 138.88 85.31) (width 0.5) (layer "F.Cu") (net 2))
   (segment (start 145.15 94.15) (end 147.815 91.485) (width 0.5) (layer "F.Cu") (net 2))
   (segment (start 127.58 94.15) (end 138.41 94.15) (width 0.5) (layer "F.Cu") (net 2))
-  (segment (start 140.98 85.31) (end 141.61 85.94) (width 0.5) (layer "F.Cu") (net 2))
   (segment (start 145.15 94.15) (end 138.41 94.15) (width 0.5) (layer "F.Cu") (net 2))
   (segment (start 138.41 94.15) (end 138.465 94.095) (width 0.5) (layer "F.Cu") (net 2))
   (segment (start 124.16 94.15) (end 127.58 94.15) (width 0.5) (layer "F.Cu") (net 2))
   (segment (start 146.48 95.48) (end 165.22 95.48) (width 0.5) (layer "F.Cu") (net 2))
-  (segment (start 141.800126 86.130126) (end 141.61 85.94) (width 0.2) (layer "F.Cu") (net 2))
   (segment (start 165.22 90.48) (end 163.54 88.8) (width 0.5) (layer "F.Cu") (net 2))
   (segment (start 154.83 57.21) (end 154.83 66.428592) (width 0.5) (layer "F.Cu") (net 3))
@@
   (segment (start 152.895 88.6) (end 152.895 87.397919) (width 0.5) (layer "F.Cu") (net 4))
   (segment (start 152.895 87.397919) (end 149.987081 84.49) (width 0.5) (layer "F.Cu") (net 4))
-  (segment (start 142.300252 87.3816) (end 142.300252 85.759748) (width 0.2) (layer "F.Cu") (net 4))
   (segment (start 153.370374 88.124626) (end 152.895 88.6) (width 0.5) (layer "F.Cu") (net 4))
-  (segment (start 141.99 85.31) (end 142.37 85.69) (width 0.5) (layer "F.Cu") (net 4))
   (segment (start 123.64 84.44) (end 141.99 84.44) (width 0.5) (layer "F.Cu") (net 4))
   (segment (start 158.175 93.88) (end 163.54 93.88) (width 0.5) (layer "F.Cu") (net 4))
-  (segment (start 142.300252 85.759748) (end 142.37 85.69) (width 0.2) (layer "F.Cu") (net 4))
   (segment (start 142.04 84.49) (end 141.99 84.44) (width 0.5) (layer "F.Cu") (net 4))
   (segment (start 121.81 82.61) (end 123.64 84.44) (width 0.5) (layer "F.Cu") (net 4))
