File: Kicad_esp_maitre_salle_blanche/Kicad_esp_maitre_salle_blanche/Kicad_esp_maitre_salle_blanche.kicad_sch (KiCad schematic)
At the start: 7 parts, among them J1 Conn_01x05_Pin, J2 Conn_01x04_Pin, U2 TLV75533PDYDR, U3 SHT40-CD1B-R3

Commit message: la carte fille "fonctionne" il serait bien de faire 2 3 changement
Parts:
- U3: footprint Esp:U_SHT3_SEN -> SHT40VRAI:SHT40-CD1B-R3_SEN
Changed lines of the file:
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@@
       (effects (font (size 1.524 1.524)))
     )
-    (property "Footprint" "Esp:U_SHT3_SEN" (at 134.62 44.45 0)
+    (property "Footprint" "SHT40VRAI:SHT40-CD1B-R3_SEN" (at 134.62 44.45 0)
       (effects (font (size 1.27 1.27) italic) hide)
     )
