File: Kicad/V1_cartebis/V1_cartebis.kicad_pcb (KiCad board)
At the start: 2 copper layers, 79 parts, among them J1 Conn_01x05_Pin, J10 Conn_01x02_Pin, J11 Conn_01x02_Pin, J12 Conn_01x02_Pin, J13 Conn_01x02_Pin, J14 Conn_01x02_Pin, J15 Conn_01x02_Pin, J16 Conn_01x02_Pin, J17 Conn_01x02_Pin, J18 Conn_01x02_Pin, J19 Conn_01x02_Pin, J2 Conn_01x02_Pin, J20 Conn_01x02_Pin, J21 Conn_01x02_Pin, J22 Conn_01x02_Pin, J23 Conn_01x02_Pin, J24 Conn_01x02_Pin, J25 Conn_01x02_Pin, J26 Conn_01x02_Pin, J27 Conn_01x02_Pin, J28 Conn_01x02_Pin, J29 Conn_01x02_Pin, J3 Conn_01x02_Pin, J30 Conn_01x02_Pin, J31 Conn_01x02_Pin, J32 Conn_01x05_Pin, J33 Conn_01x01_Pin, J34 Conn_01x01_Pin, J35 Conn_01x01_Pin, J36 Conn_01x03_Pin, J37 Conn_01x03_Pin, J38 Conn_01x03_Pin, J39 Conn_01x03_Pin, J4 Conn_01x02_Pin, J40 Conn_01x01_Pin, J41 Conn_01x01_Pin, J42 Conn_01x01_Pin, J5 Conn_01x02_Pin, J6 Conn_01x02_Pin, J7 Conn_01x02_Pin, J8 Conn_01x02_Pin, J9 Conn_01x02_Pin, U1 MCP23020-E/SO, U10 ISOM11600DFGR, U11 ISOM11600DFGR, U12 ISOM11600DFGR, U13 ISOM11600DFGR, U14 ISOM11600DFGR, U15 ISOM11600DFGR, U16 ISOM11600DFGR, U17 ISOM11600DFGR, U18 P82B715DRG4, U2 LTC24127CUHF-TRPBF, U3 ISOM11600DFGR, U4 ISOM11600DFGR, U5 ISOM11600DFGR, U6 ISOM11600DFGR, U7 ISOM11600DFGR, U8 ISOM11600DFGR, U9 ISOM11600DFGR

Commit message: la carte fille "fonctionne" il serait bien de faire 2 3 changement
Connections:
- J36 pad 1: Net-(J36-Pin_1) -> GND
- J36 pad 2: Net-(J36-Pin_1) -> GND
- J36 pad 3: Net-(J36-Pin_1) -> GND
Routing:
- net +3.3V: track 144.0 -> 156.8 mm
Changed lines of the file:
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@@
   (net 63 "Net-(J34-Pin_1)")
   (net 64 "Net-(J35-Pin_1)")
-  (net 65 "Net-(J36-Pin_1)")
-  (net 66 "Net-(J40-Pin_1)")
-  (net 67 "Net-(J41-Pin_1)")
-  (net 68 "Net-(J42-Pin_1)")
+  (net 65 "Net-(J40-Pin_1)")
+  (net 66 "Net-(J41-Pin_1)")
+  (net 67 "Net-(J42-Pin_1)")
   (footprint "Connector_PinHeader_2.54mm:PinHeader_1x02_P2.54mm_Vertical" (layer "F.Cu")
     (at 202.395 63.1 90)
@@
       (stroke (width 0.1) (type solid)) (layer "F.Fab"))
     (pad "1" thru_hole rect (at 0 0) (size 0.85 0.85) (drill 0.5) (layers "*.Cu" "*.Mask")
-      (net 67 "Net-(J41-Pin_1)") (pinfunction "Pin_1") (pintype "passive"))
+      (net 66 "Net-(J41-Pin_1)") (pinfunction "Pin_1") (pintype "passive"))
     (model "${KICAD6_3DMODEL_DIR}/Connector_PinHeader_1.00mm.3dshapes/PinHeader_1x01_P1.00mm_Vertical.wrl"
       (offset (xyz 0 0 0))
@@
       (stroke (width 0.1) (type solid)) (layer "F.Fab"))
     (pad "1" thru_hole rect (at 0 0 90) (size 0.85 0.85) (drill 0.5) (layers "*.Cu" "*.Mask")
-      (net 65 "Net-(J36-Pin_1)") (pinfunction "Pin_1") (pintype "passive"))
+      (net 1 "GND") (pinfunction "Pin_1") (pintype "passive"))
     (pad "2" thru_hole oval (at 0 1 90) (size 0.85 0.85) (drill 0.5) (layers "*.Cu" "*.Mask")
-      (net 65 "Net-(J36-Pin_1)") (pinfunction "Pin_2") (pintype "passive"))
+      (net 1 "GND") (pinfunction "Pin_2") (pintype "passive"))
     (pad "3" thru_hole oval (at 0 2 90) (size 0.85 0.85) (drill 0.5) (layers "*.Cu" "*.Mask")
-      (net 65 "Net-(J36-Pin_1)") (pinfunction "Pin_3") (pintype "passive"))
+      (net 1 "GND") (pinfunction "Pin_3") (pintype "passive"))
     (model "${KICAD6_3DMODEL_DIR}/Connector_PinHeader_1.00mm.3dshapes/PinHeader_1x03_P1.00mm_Vertical.wrl"
       (offset (xyz 0 0 0))
@@
       (stroke (width 0.1) (type solid)) (layer "F.Fab"))
     (pad "1" thru_hole rect (at 0 0) (size 0.85 0.85) (drill 0.5) (layers "*.Cu" "*.Mask")
-      (net 66 "Net-(J40-Pin_1)") (pinfunction "Pin_1") (pintype "passive"))
+      (net 65 "Net-(J40-Pin_1)") (pinfunction "Pin_1") (pintype "passive"))
     (model "${KICAD6_3DMODEL_DIR}/Connector_PinHeader_1.00mm.3dshapes/PinHeader_1x01_P1.00mm_Vertical.wrl"
       (offset (xyz 0 0 0))
@@
       (net 43 "unconnected-(U1-NC-Pad14)") (pinfunction "NC") (pintype "unspecified+no_connect"))
     (pad "15" smd rect (at 4.515 8.255 270) (size 1.9812 0.5588) (layers "F.Cu" "F.Paste" "F.Mask")
-      (net 68 "Net-(J42-Pin_1)") (pinfunction "A0") (pintype "unspecified"))
+      (net 67 "Net-(J42-Pin_1)") (pinfunction "A0") (pintype "unspecified"))
     (pad "16" smd rect (at 4.515 6.985 270) (size 1.9812 0.5588) (layers "F.Cu" "F.Paste" "F.Mask")
-      (net 67 "Net-(J41-Pin_1)") (pinfunction "A1") (pintype "unspecified"))
+      (net 66 "Net-(J41-Pin_1)") (pinfunction "A1") (pintype "unspecified"))
     (pad "17" smd rect (at 4.515 5.715 270) (size 1.9812 0.5588) (layers "F.Cu" "F.Paste" "F.Mask")
-      (net 66 "Net-(J40-Pin_1)") (pinfunction "A2") (pintype "unspecified"))
+      (net 65 "Net-(J40-Pin_1)") (pinfunction "A2") (pintype "unspecified"))
     (pad "18" smd rect (at 4.515 4.445 270) (size 1.9812 0.5588) (layers "F.Cu" "F.Paste" "F.Mask")
       (net 2 "+3.3V") (pinfunction "*RESET") (pintype "unspecified"))
@@
       (stroke (width 0.1) (type solid)) (layer "F.Fab"))
     (pad "1" thru_hole rect (at 0 0) (size 0.85 0.85) (drill 0.5) (layers "*.Cu" "*.Mask")
-      (net 68 "Net-(J42-Pin_1)") (pinfunction "Pin_1") (pintype "passive"))
+      (net 67 "Net-(J42-Pin_1)") (pinfunction "Pin_1") (pintype "passive"))
     (model "${KICAD6_3DMODEL_DIR}/Connector_PinHeader_1.00mm.3dshapes/PinHeader_1x01_P1.00mm_Vertical.wrl"
       (offset (xyz 0 0 0))
@@
   (via (at 180.59 91.4) (size 0.6) (drill 0.3) (layers "F.Cu" "B.Cu") (free) (net 1))
   (via (at 180.81 95.6) (size 0.6) (drill 0.3) (layers "F.Cu" "B.Cu") (free) (net 1))
+  (segment (start 163.73 99.45) (end 162.88 98.6) (width 0.7) (layer "F.Cu") (net 2))
   (segment (start 170.905 67.795) (end 170.91 67.79) (width 0.7) (layer "F.Cu") (net 2))
   (segment (start 171.13 52.357208) (end 171.13 62.877208) (width 0.7) (layer "F.Cu") (net 2))
@@
   (segment (start 164.377598 62.7024) (end 163.877599 62.7024) (width 0.2) (layer "F.Cu") (net 2))
   (segment (start 171.14 44.33) (end 171.14 44.5) (width 0.7) (layer "F.Cu") (net 2))
+  (segment (start 165.57 88.19) (end 165.57 89.19) (width 0.2) (layer "F.Cu") (net 2))
   (segment (start 172.38 51.107208) (end 171.13 52.357208) (width 0.7) (layer "F.Cu") (net 2))
   (segment (start 168.15 81.42) (end 168.15 78.14) (width 0.7) (layer "F.Cu") (net 2))
@@
   (segment (start 172.38 43.09) (end 172.38 51.107208) (width 0.7) (layer "F.Cu") (net 2))
   (segment (start 170.905 68.895) (end 170.905 66.045) (width 0.7) (layer "F.Cu") (net 2))
+  (segment (start 165.57 89.19) (end 165.57 90.19) (width 0.2) (layer "F.Cu") (net 2))
   (segment (start 172.88 42.59) (end 172.38 43.09) (width 0.7) (layer "F.Cu") (net 2))
   (segment (start 171.13 62.877208) (end 170.69 63.317208) (width 0.7) (layer "F.Cu") (net 2))
+  (segment (start 165.57 93.98) (end 165.57 90.19) (width 0.7) (layer "F.Cu") (net 2))
   (segment (start 164.675 64.555) (end 163.877599 63.757599) (width 0.2) (layer "F.Cu") (net 2))
+  (segment (start 162.88 98.6) (end 162.88 96.67) (width 0.7) (layer "F.Cu") (net 2))
+  (segment (start 162.88 96.67) (end 165.57 93.98) (width 0.7) (layer "F.Cu") (net 2))
   (segment (start 170.57 44.9) (end 172.88 42.59) (width 0.7) (layer "F.Cu") (net 2))
   (via (at 164.675 64.555) (size 0.6) (drill 0.3) (layers "F.Cu" "B.Cu") (net 2))
@@
   (segment (start 166.748087 59.249999) (end 168.288086 57.71) (width 0.2) (layer "F.Cu") (net 64))
   (segment (start 166.08 59.249999) (end 166.748087 59.249999) (width 0.2) (layer "F.Cu") (net 64))
-  (segment (start 167.095 83.295) (end 167.095 77.925) (width 0.7) (layer "F.Cu") (net 66))
-  (segment (start 165.17 85.22) (end 167.095 83.295) (width 0.7) (layer "F.Cu") (net 66))
-  (segment (start 166.155 78.255) (end 165.825 77.925) (width 0.7) (layer "F.Cu") (net 67))
-  (segment (start 165.825 77.925) (end 165.825 78.6362) (width 0.2) (layer "F.Cu") (net 67))
-  (segment (start 166.155 82.215) (end 166.155 78.255) (width 0.7) (layer "F.Cu") (net 67))
-  (segment (start 165.825 78.6362) (end 166.18 78.9912) (width 0.2) (layer "F.Cu") (net 67))
-  (segment (start 165.16 83.21) (end 166.155 82.215) (width 0.7) (layer "F.Cu") (net 67))
-  (segment (start 165.18 81.17) (end 164.555 80.545) (width 0.7) (layer "F.Cu") (net 68))
-  (segment (start 164.555 80.545) (end 164.555 77.925) (width 0.7) (layer "F.Cu") (net 68))
+  (segment (start 167.095 83.295) (end 167.095 77.925) (width 0.7) (layer "F.Cu") (net 65))
+  (segment (start 165.17 85.22) (end 167.095 83.295) (width 0.7) (layer "F.Cu") (net 65))
+  (segment (start 166.155 78.255) (end 165.825 77.925) (width 0.7) (layer "F.Cu") (net 66))
+  (segment (start 165.825 77.925) (end 165.825 78.6362) (width 0.2) (layer "F.Cu") (net 66))
+  (segment (start 166.155 82.215) (end 166.155 78.255) (width 0.7) (layer "F.Cu") (net 66))
+  (segment (start 165.825 78.6362) (end 166.18 78.9912) (width 0.2) (layer "F.Cu") (net 66))
+  (segment (start 165.16 83.21) (end 166.155 82.215) (width 0.7) (layer "F.Cu") (net 66))
+  (segment (start 165.18 81.17) (end 164.555 80.545) (width 0.7) (layer "F.Cu") (net 67))
+  (segment (start 164.555 80.545) (end 164.555 77.925) (width 0.7) (layer "F.Cu") (net 67))
   (zone (net 1) (net_name "GND") (layers "F&B.Cu") (hatch edge 0.5)
     (connect_pads (clearance 0.5))
