File: Kicad/V1_cartebis/V1_cartebis.kicad_sch (KiCad schematic)
At the start: 17 parts, among them J1 Conn_01x05_Pin, J32 Conn_01x05_Pin, J33 Conn_01x01_Pin, J34 Conn_01x01_Pin, J35 Conn_01x01_Pin, J36 Conn_01x03_Pin, J37 Conn_01x03_Pin, J38 Conn_01x03_Pin, J39 Conn_01x03_Pin, J40 Conn_01x01_Pin, J41 Conn_01x01_Pin, J42 Conn_01x01_Pin, U1 MCP23020-E/SO, U18 P82B715DRG4, U2 LTC24127CUHF-TRPBF

Commit message: la carte fille "fonctionne" il serait bien de faire 2 3 changement
Connections:
- net GND: now also J36.1 (Pin_1), J36.2 (Pin_2), J36.3 (Pin_3)
Changed lines of the file:
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@@
   (junction (at 225.044 21.082) (diameter 0) (color 0 0 0 0)
+  )
+  (junction (at 234.95 21.336) (diameter 0) (color 0 0 0 0)
   )
   (junction (at 121.92 95.758) (diameter 0) (color 0 0 0 0)
@@
   )
   (junction (at 225.044 18.542) (diameter 0) (color 0 0 0 0)
-  )
-  (junction (at 234.95 21.336) (diameter 0) (color 0 0 0 0)
   )
   (junction (at 243.84 18.796) (diameter 0) (color 0 0 0 0)
@@
     (stroke (width 0) (type default))
   )
-  (wire (pts (xy 234.95 21.59) (xy 234.95 23.114))
+  (wire (pts (xy 234.95 21.336) (xy 234.95 23.114))
     (stroke (width 0) (type default))
   )
@@
     (stroke (width 0) (type default))
   )
+  (wire (pts (xy 243.84 21.336) (xy 243.84 22.606))
+    (stroke (width 0) (type default))
+  )
   (wire (pts (xy 234.95 18.796) (xy 234.95 21.336))
     (stroke (width 0) (type default))
   )
-  (wire (pts (xy 234.696 21.336) (xy 234.95 21.336))
-    (stroke (width 0) (type default))
-  )
-  (wire (pts (xy 243.84 21.336) (xy 243.84 22.606))
-    (stroke (width 0) (type default))
-  )
